File: SMD_test/SMD_test.kicad_pcb (KiCad board)
At the start: 4 copper layers, 46 x 49.4 mm, 7 parts, among them J1 Conn_01x03_Pin

Commit message: updated SMD_test
Parts:
- A1, C1, D1, J1, R1, R2: moved to B.Cu
- moved C1 54.5 mm to (163.6, 123.3)
- moved D1 50.2 mm to (161.4, 109.9), turned to 180 degrees
- moved R1 44.2 mm to (158.4, 124.4)
- moved A1 36.7 mm to (154.6, 82.3), turned to 180 degrees
- moved R2 20.2 mm to (126.6, 112.6), turned to 0 degrees
- moved G*** 18.3 mm to (144.6, 99.2)
- moved J1 14.6 mm to (129.5, 91.7), turned to 180 degrees
Other:
- outline, holes or cut-outs redrawn

Commit message: updated SMD_test
Other:
- board text added: "im nayeon! yoo jeongyeon! momo-jjang! sana-jjang! park jihyo! mina-jjang! kim dahyun! son chaeyoung! chou tzuyu! won ineo millieon! sesange dan hanappunin teu.wa.i.seu"
Changed lines of the file:
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@@
 			(plotvalue yes)
 			(plotfptext yes)
-			(plotinvisibletext no)
+			(plotinvisibletext yes)
 			(sketchpadsonfab no)
 			(subtractmaskfromsilk no)
@@
 	)
 	(gr_text "Carson\n"
-		(at 167.46 78.97 -0)
-		(layer "B.Cu")
+		(at 167.46 78.97 0)
+		(layer "B.SilkS")
 		(effects
 			(font
@@
 	)
 	(gr_text "v1.0"
-		(at 130.16 122.77 -0)
-		(layer "B.Cu")
+		(at 130.16 122.77 0)
+		(layer "B.SilkS")
 		(effects
 			(font
@@
 	)
 	(gr_text "07/SEPT/\n2026"
-		(at 137.06 122.87 -0)
-		(layer "B.Cu")
+		(at 137.06 122.87 0)
+		(layer "B.SilkS")
 		(effects
 			(font
@@
 	)
 	(gr_text "Wu\n"
-		(at 167.06 81.27 -0)
-		(layer "B.Cu")
+		(at 167.06 81.27 0)
+		(layer "B.SilkS")
 		(effects
 			(font
@@
 		)
 	)
-	(gr_text "SMD Test"
-		(at 137.06 118.07 -0)
-		(layer "B.Cu")
+	(gr_text "im nayeon! \nyoo jeongyeon! \nmomo-jjang! \nsana-jjang!\npark jihyo! \nmina-jjang! \nkim dahyun! \nson chaeyoung! \nchou tzuyu!\nwon ineo millieon! \nsesange dan hanappunin \nteu.wa.i.seu"
+		(at 167.1 91.4 0)
+		(layer "B.SilkS")
 		(effects
 			(font
+				(size 0.5 0.5)
+				(thickness 0.05)
+				(bold yes)
+			)
+			(justify left bottom mirror)
+		)
+	)
+	(gr_text "SMD Test"
+		(at 137.06 118.07 0)
+		(layer "B.SilkS")
+		(effects
+			(font

Commit message: updated SMD_test
Other:
- board text added: "A1"
- board text added: "C1"
- board text added: "D1"
- board text added: "J1"
- board text added: "R1"
- board text added: "R2"
- board text removed: "im nayeon! yoo jeongyeon! momo-jjang! sana-jjang! park jihyo! mina-jjang! kim dahyun! son chaeyoung! chou tzuyu! won ineo millieon! sesange dan hanappunin teu.wa.i.seu"
Changed lines of the file:
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@@
 		(layer "Edge.Cuts")
+	)
+	(gr_text "R1\n"
+		(at 158.8 119.7 90)
+		(layer "B.SilkS")
+		(effects
+			(font
+				(size 0.8128 0.8128)
+				(thickness 0.1524)
+				(bold yes)
+			)
+			(justify left bottom mirror)
+		)
+	)
+	(gr_text "J1"
+		(at 130 93 0)
+		(layer "B.SilkS")
+		(effects
+			(font
+				(size 0.8128 0.8128)
+				(thickness 0.1524)
+				(bold yes)
+			)
+			(justify left bottom mirror)
+		)
 	)
 	(gr_text "Carson\n"
@@
 				(size 1.524 1.524)
 				(thickness 0.3048)
+				(bold yes)
+			)
+			(justify left bottom mirror)
+		)
+	)
+	(gr_text "D1"
+		(at 165.1 110.4 0)
+		(layer "B.SilkS")
+		(effects
+			(font
+				(size 0.8128 0.8128)
+				(thickness 0.1524)
 				(bold yes)
 			)
@@
 		)
 	)
-	(gr_text "im nayeon! \nyoo jeongyeon! \nmomo-jjang! \nsana-jjang!\npark jihyo! \nmina-jjang! \nkim dahyun! \nson chaeyoung! \nchou tzuyu!\nwon ineo millieon! \nsesange dan hanappunin \nteu.wa.i.seu"
-		(at 167.1 91.4 0)
+	(gr_text "A1"
+		(at 147.9 98.6 0)
 		(layer "B.SilkS")
 		(effects
 			(font
-				(size 0.5 0.5)
-				(thickness 0.05)
+				(size 0.8128 0.8128)
+				(thickness 0.1524)
+				(bold yes)
+			)
+			(justify left bottom mirror)
+		)
+	)
+	(gr_text "C1\n"
+		(at 164.2 119.9 90)
+		(layer "B.SilkS")
+		(effects
+			(font
+				(size 0.8128 0.8128)
+				(thickness 0.1524)
 				(bold yes)
 			)
@@
 				(bold yes)
 			)
+			(justify left bottom mirror)
+		)
+	)
+	(gr_text "R2"
+		(at 131.4 113.1 0)
+		(layer "B.SilkS")
+		(effects
+			(font
+				(size 0.8128 0.8128)
+				(thickness 0.1524)
+				(bold yes)
+			)

Commit message: updated SMD_test
Other:
- board text added: "Twicetagram Eyes Wide Open Formula of Love: O+T=<3 This Is For Ten: The Story Goes On"
Changed lines of the file:
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@@
+		)
+	)
+	(gr_text "Twicetagram\nEyes Wide Open\nFormula of Love: \nO+T=<3\nThis Is For\nTen: The Story \nGoes On"
+		(at 167.2 90.7 0)
+		(layer "B.SilkS")
+		(effects
+			(font
+				(size 0.8128 0.8128)
+				(thickness 0.1524)
+				(bold yes)
+			)
+			(justify left bottom mirror)
 		)
 	)
