File: Tamagotchi/CAD/Tamagotchi/Tamagotchi.kicad_pcb (KiCad board)
At the start: 2 copper layers, 17 parts, among them J1 Conn_01x02_Pin, SW1 SW_Push, SW2 SW_Push, SW3 SW_Push, SW4 SW_Push, SW5 SW_SPDT, U1 ESP32-C3-SuperMini

Commit message: updated Tamagotchi
Parts:
- added U2: SSD1306, spo2_stuff:SSD1306, F.Cu at (135.2, 70.9)
- moved SW5 46.3 mm to (154.2, 62.9)
- moved J1 40.5 mm to (152.5, 75.6)
- moved SW1 35.9 mm to (112.6, 61.4)
- moved SW2 35.9 mm to (112.6, 70.0)
- moved SW3 35.9 mm to (112.6, 78.5)
- moved SW4 35.9 mm to (112.6, 87.1)
- moved D1 34.7 mm to (152.7, 69.6)
- moved R1 21.2 mm to (143.2, 91.0)
- moved R2 21.2 mm to (143.2, 95.1)
- moved R3 21.2 mm to (143.2, 99.1)
- moved R4 21.2 mm to (143.2, 103.2)
- moved R5 21.2 mm to (143.2, 107.2)
- moved U1 16.9 mm to (131.4, 101.5)
- moved C1 4.21 mm to (154.0, 91.0)
- moved C2 4.21 mm to (154.0, 95.1)
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Connections:
- U1 pad 3V3: (no net) -> Net-(SW5-C)
- U1 pad 5V: (no net) -> unconnected-(U1-Pad5V)
- U1 pad GND: (no net) -> GND

Commit message: updated Tamagotchi
Parts:
- added BT1: Battery_Cell, Connector_PinHeader_2.54mm:PinHeader_1x02_P2.54mm_Vertical, F.Cu at (152.5, 90.1)
- J1: value Conn_01x02_Pin -> Conn_01x06_Pin; footprint Connector_PinHeader_2.54mm:PinHeader_1x02_P2.54mm_Vertical -> Connector_PinHeader_2.54mm:PinHeader_1x06_P2.54mm_Vertical
- moved D1 46.1 mm to (154.7, 115.6)
- moved C1 24.1 mm to (151.6, 67.0)
- moved C2 24.1 mm to (151.6, 71.1)
- moved C3 24.1 mm to (151.6, 75.1)
- moved C4 24.1 mm to (151.6, 79.2)
- moved SW5 21.8 mm to (154.0, 84.7)
- moved J1 21.4 mm to (154.5, 96.9)
- moved R4 5.62 mm to (143.0, 108.8)
- moved R5 5.62 mm to (143.0, 112.8)
- moved SW1 5.62 mm to (112.4, 67.0)
- moved SW2 5.62 mm to (112.4, 75.6)
- moved U1 5.62 mm to (131.2, 107.1)
- moved R1 5.62 mm to (143.0, 96.6)
- moved R2 5.62 mm to (143.0, 100.7)
- moved R3 5.62 mm to (143.0, 104.7)
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
Commit message: updated Tamagotchi
Parts:
- moved D1 58.0 mm to (111.2, 77.2)
- moved R4 52.9 mm to (113.2, 65.0), turned to -90 degrees
- moved SW3 47.8 mm to (160.2, 86.7)
- moved SW2 47.8 mm to (160.2, 76.7)
- moved SW1 47.8 mm to (160.2, 66.5)
- moved R5 40.2 mm to (118.0, 81.3), turned to 90 degrees
- moved J1 40.1 mm to (116.1, 85.2), turned to -90 degrees
- moved C4 34.5 mm to (118.0, 71.2), turned to 90 degrees
- moved R1 34.5 mm to (157.0, 65.1), turned to -90 degrees
- moved R2 29.3 mm to (157.0, 74.9), turned to -90 degrees
- moved SW4 28.0 mm to (103.2, 66.2)
- moved R3 24.3 mm to (157.0, 84.8), turned to -90 degrees
- moved C3 15.9 mm to (152.4, 91.0), turned to 90 degrees
- moved BT1 14.7 mm to (165.5, 97.0)
- moved SW5 12.6 mm to (152.8, 97.2)
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
Commit message: updated Tamagotchi
Parts:
- removed BT1: Battery_Cell, Connector_PinHeader_2.54mm:PinHeader_1x02_P2.54mm_Vertical
- moved SW4 69.5 mm to (160.2, 106.0)
- moved R4 58.6 mm to (157.0, 104.0)
- moved C4 51.7 mm to (152.2, 110.0)
- moved D1 41.1 mm to (138.5, 108.0)
- moved R5 33.6 mm to (132.5, 111.6)
- moved U1 26.3 mm to (110.4, 104.4)
- moved J1 15.3 mm to (102.2, 91.8), turned to 90 degrees
- moved SW5 14.5 mm to (138.4, 98.5), turned to 180 degrees
- moved C3 5.80 mm to (152.4, 96.8)
- moved R3 5.80 mm to (157.0, 90.6)
- moved SW3 5.80 mm to (160.2, 92.5)
- moved C2 3.30 mm to (152.4, 84.1)
- moved R2 3.30 mm to (157.0, 78.2)
- moved SW2 3.30 mm to (160.2, 80.0)
Routing:
- added copper zone on F.Cu, net (none)
Other:
- board outline added: 73.8 x 52.5 mm

Commit message: updated Tamagotchi
Parts:
- moved J1 30.3 mm to (114.3, 64.0), turned to -90 degrees
- moved U1 2.64 mm to (107.9, 105.1), turned to 0 degrees
- moved D1 2.29 mm to (140.8, 108.0), turned to 180 degrees
- moved SW5 0.15 mm to (138.2, 98.5)
Routing:
- net Net-(SW5-C): track 0.00 -> 128.8 mm, vias 0 -> 3
- net Net-(U1-GPIO0): track 0.00 -> 80.1 mm
- net Net-(U1-GPIO1): track 0.00 -> 72.9 mm
- net Net-(U1-GPIO2): track 0.00 -> 61.7 mm
- net Net-(U1-GPIO8): track 0.00 -> 61.6 mm
- net Net-(J1-Pin_1): track 0.00 -> 60.2 mm
- net Net-(U1-GPIO9): track 0.00 -> 59.1 mm
- net Net-(U1-GPIO3): track 0.00 -> 56.1 mm
- net Net-(U1-GPIO4): track 0.00 -> 20.2 mm
- net Net-(D1-A): track 0.00 -> 7.37 mm
- added copper zone on F.Cu, net GND
- removed copper zone on F.Cu, net (none)
Other:
- board size 73.8 x 52.5 mm -> 73.8 x 55 mm
- board text added: "Carson Wu"
- board text added: "JLCJLCJLCJLC"
- board text added: "Tamagotchi"
- board text added: "v1.0 - 14/SEPT/2026"

Commit message: updated Tamagotchi
Other:
- board text added: "v1.1 - 14/SEPT/2026"
- board text removed: "v1.0 - 14/SEPT/2026"

Commit message: updated Tamagotchi
Parts:
- moved J1 0.45 mm to (114.8, 64.0)
Other:
- board text added: "v1.1 14/SEPT/2026"
- board text removed: "v1.1 - 14/SEPT/2026"
