File: muichiro_desk_lamp/muichiro_desk_lamp.kicad_sch (KiCad schematic)
At the start: 6 parts, among them J1 Conn_01x03_Pin

Commit message: updated muichiro_desk_lamp
Parts:
- removed A1: Arduino_Nano_v3.x, Module:Arduino_Nano, symbol MCU_Module:Arduino_Nano_v3.x
- added U1: ESP32-C3-DevKitM-1, desk-lamp:ESP32_Socket_Dual_1x15, symbol RF_Module:ESP32-C3-DevKitM-1
- C1: footprint Capacitor_THT:C_Disc_D4.7mm_W2.5mm_P5.00mm -> Capacitor_SMD:C_0805_2012Metric
- D1: footprint LED_THT:LED_D5.0mm -> LED_SMD:LED_0805_2012Metric
- J1: footprint Library:SW-420 -> Connector_PinSocket_2.54mm:PinSocket_1x03_P2.54mm_Vertical_SMD_Pin1Left
- R1, R2: footprint Resistor_THT:R_Axial_DIN0204_L3.6mm_D1.6mm_P7.62mm_Horizontal -> Resistor_SMD:R_0805_2012Metric
Connections:
- net +5V: now also U1.13 (5V), U1.14 (5V)
- net GND: now also U1.1 (GND), U1.12 (GND), U1.15 (GND), U1.16 (GND), U1.19 (GND), U1.24 (GND), U1.27 (GND), U1.30 (GND), U1.6 (GND), U1.8 (GND)
- net at R1.1: now also U1.21 (IO5)
- net at C1.1, J1.3 (Pin_3): now also U1.5 (IO3)
- new net: U1.2 (3V3), U1.3 (3V3)
- no-connect marks 25 -> 15

Commit message: updated muichiro_desk_lamp
Parts:
- added D2, D3, D4: LED, LED_SMD:LED_0805_2012Metric, symbol Device:LED
- added R3, R4, R5: 1K, Resistor_SMD:R_0805_2012Metric, symbol Device:R
Connections:
- net +5V: no longer R2.1
- net GND: now also D2.1 (K), D3.1 (K), D4.1 (K)
- net at U1.20 (IO4): now also R3.1
- net at U1.22 (IO6): now also R4.1
- net at U1.4 (IO2): now also R5.1
- new net: D2.2 (A), R3.2
- new net: D4.2 (A), R5.2
- new net: D3.2 (A), R4.2
- new net +3V3: R2.1
- no-connect marks 15 -> 9
Other:
- moved on the sheet: D1, R1
