File: muichiro_desk_lamp/muichiro_desk_lamp.kicad_pcb (KiCad board)
At the start: 2 copper layers, 102.6 x 123.6 mm, 7 parts, among them J1 Conn_01x03_Pin, U1 ESP32-C3-DevKitM-1

Commit message: updated muichiro_desk_lamp
Parts:
- added D2: LED, LED_SMD:LED_0805_2012Metric, F.Cu at (192.9, 48.6)
- added D3: LED, LED_SMD:LED_0805_2012Metric, F.Cu at (191.8, 112.0)
- added D4: LED, LED_SMD:LED_0805_2012Metric, F.Cu at (146.1, 112.2)
- added R3: 1K, Resistor_SMD:R_0805_2012Metric, F.Cu at (188.3, 48.8)
- added R4: 1K, Resistor_SMD:R_0805_2012Metric, F.Cu at (187.1, 112.2)
- added R5: 1K, Resistor_SMD:R_0805_2012Metric, F.Cu at (141.6, 112.4)
- moved R1 54.6 mm to (142.4, 48.9)
- moved D1 53.1 mm to (147.0, 48.8)
- moved C1 19.2 mm to (186.2, 95.0)
- moved G*** 13.7 mm to (167.1, 80.5)
- moved R2 10.7 mm to (185.8, 78.0)
- moved U1 10.5 mm to (166.7, 107.0)
- moved J1 8.64 mm to (185.8, 86.5)
Connections:
- R2 pad 1: +5V -> +3V3
- U1 pad 20: unconnected-(U1-IO4-Pad20) -> Net-(U1-IO4)
- U1 pad 22: unconnected-(U1-IO6-Pad22) -> Net-(U1-IO6)
- U1 pad 4: unconnected-(U1-IO2-Pad4) -> Net-(U1-IO2)
Routing:
- net +5V: track 103.4 -> 4.35 mm
- net Net-(U1-IO2): track 0.00 -> 42.6 mm
- net GND: track 41.4 -> 0.00 mm
- net Net-(U1-IO4): track 0.00 -> 38.5 mm
- net Net-(U1-IO5): track 14.5 -> 49.7 mm
- net Net-(U1-IO6): track 0.00 -> 32.5 mm
- net Net-(J1-Pin_1): track 12.8 -> 7.04 mm
- net Net-(D3-A): track 0.00 -> 5.62 mm
- net Net-(D2-A): track 0.00 -> 5.42 mm
- net Net-(D4-A): track 0.00 -> 5.32 mm
- net Net-(D1-A): track 4.65 -> 5.38 mm
Other:
- board size 102.6 x 123.6 mm -> 58.3 x 70.7 mm
- board text added: "Capacitor (100N)"
- board text added: "ESP32-C3-DevKitM-1"
- board text added: "JLCJLCJLCJLC"
- board text added: "LED (Green)"
- board text added: "Resistor (1K)"
- board text added: "SW-420"

Commit message: updated muichiro_desk_lamp
Parts:
- C1, D1, D2, D3, D4, J1, R1, R2, R3, R4, R5, U1: moved to B.Cu
- G***: moved to F.Cu
- moved R5 51.8 mm to (193.4, 112.4), turned to 180 degrees
- moved D2 50.7 mm to (142.2, 48.6), turned to 180 degrees
- moved R1 50.2 mm to (192.6, 48.9), turned to 180 degrees
- moved D3 48.7 mm to (143.2, 112.0), turned to 180 degrees
- moved D4 42.9 mm to (189.0, 112.2), turned to 180 degrees
- moved R3 41.6 mm to (146.7, 48.8), turned to 180 degrees
- moved D1 41.1 mm to (188.1, 48.8), turned to 180 degrees
- moved R4 39.1 mm to (147.9, 112.2), turned to 180 degrees
- moved C1 37.5 mm to (148.8, 95.0), turned to 180 degrees
- moved J1 36.7 mm to (149.2, 86.5), turned to 180 degrees
- moved R2 36.6 mm to (149.2, 78.0), turned to 180 degrees
- moved U1 1.71 mm to (168.4, 107.0), turned to 180 degrees
- moved G*** 0.84 mm to (167.9, 80.4), turned to 0 degrees
Routing:
- added copper zone on B.Cu, net GND
- removed copper zone on F.Cu, net GND

Commit message: updated Tamagotchi and muichiro_desk_lamp
Other:
- board text added: "Carson Wu muichiro_desk_lamp 19/10/2026"
Changed lines of the file:
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@@
+		)
+	)
+	(gr_text "Carson Wu\nmuichiro_desk_lamp\n19/10/2026"
+		(at 180.34 57.404 0)
+		(layer "B.SilkS")
+		(effects
+			(font
+				(size 1.524 1.524)
+				(thickness 0.3048)
+				(bold yes)
+			)
+			(justify left bottom mirror)
 		)
 	)

Commit message: updated Tamagotchi and muichiro_desk_lamp
Parts:
- removed U1: ESP32-C3-DevKitM-1, desk-lamp:ESP32_Socket_Dual_1x15
- added J2: Conn_01x08_Socket, Connector_PinSocket_2.54mm:PinSocket_1x08_P2.54mm_Vertical_SMD_Pin1Left, B.Cu at (163.2, 78.2)
- added J3: Conn_01x08_Socket, Connector_PinSocket_2.54mm:PinSocket_1x08_P2.54mm_Vertical_SMD_Pin1Left, B.Cu at (178.4, 78.2)
- R1, R3, R4, R5: value 1K -> 220Ω
- moved R4 45.7 mm to (193.7, 112.3)
- moved D3 45.7 mm to (188.9, 112.1)
- moved D4 45.6 mm to (143.4, 112.1)
- moved R5 45.6 mm to (147.8, 112.3)
Routing:
- net +3V3: track 0.00 -> 34.0 mm
- net Net-(J1-Pin_3): track 43.1 -> 22.9 mm
- net Net-(J3-Pin_4): track 49.7 -> 36.2 mm
- net +5V: track 4.35 -> 0.00 mm
- net Net-(J2-Pin_4): track 42.6 -> 39.4 mm
- net Net-(J3-Pin_5): track 38.5 -> 40.8 mm
- net Net-(J3-Pin_2): track 32.5 -> 33.7 mm
Other:
- board text added: "ESP32-C3-SuperMini"
- board text added: "Resistor (220Ω)"
- board text removed: "ESP32-C3-DevKitM-1"
- board text removed: "Resistor (1K)"
