File: muichiro_desk_lamp/muichiro_desk_lamp.kicad_pcb (KiCad board)
At the start: 2 copper layers, 58.3 x 70.7 mm, 14 parts, among them J1 Conn_01x03_Pin, J2 Conn_01x08_Socket, J3 Conn_01x08_Socket

Commit message: updated Tamagotchi and muichiro_desk_lamp
Routing:
- net Net-(D1-A): track 5.30 -> 8.46 mm
- net Net-(D2-A): track 5.25 -> 8.19 mm
- net +3V3: track 34.0 -> 35.1 mm
- net Net-(D4-A): track 5.15 -> 6.07 mm
- net Net-(D3-A): track 5.45 -> 6.15 mm
Changed lines of the file:
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@@
 		(start 150.82 80.5)
 		(end 148.32 78)
-		(width 0.127)
+		(width 0.14)
 		(layer "B.Cu")
 		(net "Net-(J1-Pin_1)")
@@
 		(start 150.82 84)
 		(end 150.82 80.5)
-		(width 0.127)
+		(width 0.14)
 		(layer "B.Cu")
 		(net "Net-(J1-Pin_1)")
@@
 		(start 150.82 89.08)
 		(end 150.82 87.684)
-		(width 0.127)
+		(width 0.14)
 		(layer "B.Cu")
 		(net "Net-(J1-Pin_3)")
@@
 		(start 150.82 87.684)
 		(end 161.544 76.96)
-		(width 0.127)
+		(width 0.14)
 		(layer "B.Cu")
 		(net "Net-(J1-Pin_3)")
@@
 		(start 149.72 90.18)
 		(end 150.82 89.08)
-		(width 0.127)
+		(width 0.14)
 		(layer "B.Cu")
 		(net "Net-(J1-Pin_3)")
@@
 		(start 149.72 95)
 		(end 149.72 90.18)
-		(width 0.127)
-		(layer "B.Cu")
-		(net "Net-(J1-Pin_3)")
+		(width 0.14)
+		(layer "B.Cu")
+		(net "Net-(J1-Pin_3)")
+	)
+	(segment
+		(start 150.876 110.1325)
+		(end 150.876 94.974)
+		(width 0.14)
+		(layer "B.Cu")
+		(net "Net-(J2-Pin_4)")
+	)
+	(segment
+		(start 150.876 94.974)
+		(end 164.844 81.006)
+		(width 0.14)
+		(layer "B.Cu")
+		(net "Net-(J2-Pin_4)")
 	)
 	(segment
 		(start 164.844 81.006)
 		(end 164.844 79.5)
-		(width 0.127)
-		(layer "B.Cu")
-		(net "Net-(J2-Pin_4)")
-	)
-	(segment
-		(start 150.4105 110.598)
-		(end 150.4105 95.4395)
-		(width 0.127)
-		(layer "B.Cu")
-		(net "Net-(J2-Pin_4)")
-	)
-	(segment
-		(start 150.4105 95.4395)
-		(end 164.844 81.006)
-		(width 0.127)
+		(width 0.14)
 		(layer "B.Cu")
 		(net "Net-(J2-Pin_4)")
@@
 	(segment
 		(start 148.7405 112.268)
-		(end 150.4105 110.598)
-		(width 0.127)
-		(layer "B.Cu")
-		(net "Net-(J2-Pin_4)")
-	)
-	(segment
-		(start 146.225 112.9585)
+		(end 150.876 110.1325)
+		(width 0.14)
+		(layer "B.Cu")
+		(net "Net-(J2-Pin_4)")
+	)
+	(segment
+		(start 143.764 113.792)
+		(end 145.3915 113.792)
+		(width 0.14)
+		(layer "B.Cu")
+		(net "Net-(D4-A)")
+	)
+	(segment
+		(start 142.4155 112.068)
+		(end 142.4155 112.4435)
+		(width 0.14)
+		(layer "B.Cu")
+		(net "Net-(D4-A)")
+	)
+	(segment
+		(start 142.4155 112.4435)
+		(end 143.764 113.792)
+		(width 0.14)
+		(layer "B.Cu")
+		(net "Net-(D4-A)")
+	)
+	(segment
+		(start 145.3915 113.792)
 		(end 146.9155 112.268)
-		(width 0.127)
-		(layer "B.Cu")
-		(net "Net-(D4-A)")
-	)
-	(segment
-		(start 143.306 112.9585)
-		(end 146.225 112.9585)
-		(width 0.127)
-		(layer "B.Cu")
-		(net "Net-(D4-A)")
-	)
-	(segment
-		(start 142.4155 112.068)
-		(end 143.306 112.9585)
-		(width 0.127)
-		(layer "B.Cu")
-		(net "Net-(D4-A)")
-	)
-	(segment
-		(start 142.1105 49.4905)
-		(end 145.1295 49.4905)
-		(width 0.127)
+		(width 0.14)
+		(layer "B.Cu")
+		(net "Net-(D4-A)")
+	)
+	(segment
+		(start 141.22 50.288)
+		(end 141.732 50.8)
+		(width 0.14)
+		(layer "B.Cu")
+		(net "Net-(D2-A)")
+	)
+	(segment
+		(start 145.288 50.8)
+		(end 145.82 50.268)
+		(width 0.14)
 		(layer "B.Cu")
 		(net "Net-(D2-A)")
@@
 	(segment
 		(start 141.22 48.6)
-		(end 142.1105 49.4905)
-		(width 0.127)
-		(layer "B.Cu")
-		(net "Net-(D2-A)")
-	)
-	(segment
-		(start 145.1295 49.4905)
+		(end 141.22 50.288)
+		(width 0.14)
+		(layer "B.Cu")
+		(net "Net-(D2-A)")
+	)
+	(segment
+		(start 145.82 50.268)
 		(end 145.82 48.8)
-		(width 0.127)
+		(width 0.14)
+		(layer "B.Cu")
+		(net "Net-(D2-A)")
+	)
+	(segment
+		(start 141.732 50.8)
+		(end 145.288 50.8)
+		(width 0.14)
 		(layer "B.Cu")
 		(net "Net-(D2-A)")
@@
 		(start 193.545 62.798)
 		(end 180.09 76.253)
-		(width 0.127)
+		(width 0.14)
 		(layer "B.Cu")
 		(net "Net-(J3-Pin_4)")
@@
 		(start 193.545 48.9)
 		(end 193.545 62.798)
-		(width 0.127)
+		(width 0.14)
 		(layer "B.Cu")
 		(net "Net-(J3-Pin_4)")
@@
 		(start 180.09 76.253)
 		(end 180.09 79.502)
-		(width 0.127)
+		(width 0.14)
 		(layer "B.Cu")
 		(net "Net-(J3-Pin_4)")
 	)
 	(segment
-		(start 188.0105 49.6905)
-		(end 190.9295 49.6905)
-		(width 0.127)
-		(layer "B.Cu")
-		(net "Net-(D1-A)")
-	)
-	(segment
-		(start 190.9295 49.6905)
+		(start 187.12 50.468)
+		(end 187.788 51.136)
+		(width 0.14)
+		(layer "B.Cu")
+		(net "Net-(D1-A)")
+	)
+	(segment
+		(start 191.18 51.136)
+		(end 191.72 50.596)
+		(width 0.14)
+		(layer "B.Cu")
+		(net "Net-(D1-A)")
+	)
+	(segment
+		(start 187.12 48.8)
+		(end 187.12 50.468)
+		(width 0.14)
+		(layer "B.Cu")
+		(net "Net-(D1-A)")
+	)
+	(segment
+		(start 191.72 50.596)
 		(end 191.72 48.9)
-		(width 0.127)
-		(layer "B.Cu")
-		(net "Net-(D1-A)")
-	)
-	(segment
-		(start 187.12 48.8)
-		(end 188.0105 49.6905)
-		(width 0.127)
-		(layer "B.Cu")
-		(net "Net-(D1-A)")
-	)
-	(segment
-		(start 192.0485 112.9585)
+		(width 0.14)
+		(layer "B.Cu")
+		(net "Net-(D1-A)")
+	)
+	(segment
+		(start 187.788 51.136)
+		(end 191.18 51.136)
+		(width 0.14)
+		(layer "B.Cu")
+		(net "Net-(D1-A)")
+	)
+	(segment
+		(start 191.215 113.792)
 		(end 192.739 112.268)
-		(width 0.127)
+		(width 0.14)
 		(layer "B.Cu")
 		(net "Net-(D3-A)")
 	)
 	(segment
-		(start 188.8295 112.9585)
-		(end 192.0485 112.9585)
-		(width 0.127)
+		(start 187.939 112.068)
+		(end 189.663 113.792)
+		(width 0.14)
 		(layer "B.Cu")
 		(net "Net-(D3-A)")
 	)
 	(segment
-		(start 187.939 112.068)
-		(end 188.8295 112.9585)
-		(width 0.127)
+		(start 189.663 113.792)
+		(end 191.215 113.792)
+		(width 0.14)
 		(layer "B.Cu")
 		(net "Net-(D3-A)")
@@
 		(start 194.564 99.056)
 		(end 180.09 84.582)
-		(width 0.127)
+		(width 0.14)
 		(layer "B.Cu")
 		(net "Net-(J3-Pin_2)")
@@
 		(start 194.564 112.268)
 		(end 194.564 99.056)
-		(width 0.127)
+		(width 0.14)
 		(layer "B.Cu")
 		(net "Net-(J3-Pin_2)")
@@
 		(start 147.645 48.8)
 		(end 148.628 48.8)
-		(width 0.127)
+		(width 0.14)
 		(layer "B.Cu")
 		(net "Net-(J3-Pin_5)")
@@
 		(start 148.628 48.8)
 		(end 176.79 76.962)
-		(width 0.127)
+		(width 0.14)
 		(layer "B.Cu")
 		(net "Net-(J3-Pin_5)")
 	)
 	(segment
-		(start 178.0875 77.6525)
-		(end 180.09 75.65)
-		(width 0.127)
-		(layer "B.Cu")
-		(net "+3V3")
-	)
-	(segment
-		(start 180.09 75.65)
-		(end 180.09 74.422)
-		(width 0.127)
-		(layer "B.Cu")
-		(net "+3V3")
-	)
-	(segment
-		(start 175.6495 77.6525)
-		(end 178.0875 77.6525)
-		(width 0.127)
-		(layer "B.Cu")
-		(net "+3V3")
-	)
-	(segment
-		(start 173.397 75.4)
-		(end 175.6495 77.6525)
-		(width 0.127)
-		(layer "B.Cu")
-		(net "+3V3")
-	)
-	(segment
-		(start 152.745 75.4)
-		(end 173.397 75.4)
-		(width 0.127)
+		(start 172.9125 75.4)
+		(end 176.2525 78.74)
+		(width 0.14)
 		(layer "B.Cu")
 		(net "+3V3")
@@
 		(start 150.145 78)
 		(end 152.745 75.4)
-		(width 0.127)
-		(layer "B.Cu")
-		(net "+3V3")
+		(width 0.14)
+		(layer "B.Cu")
+		(net "+3V3")
+	)
+	(segment
+		(start 180.09 75.875404)
+		(end 180.09 74.422)
+		(width 0.14)
+		(layer "B.Cu")
+		(net "+3V3")
+	)
+	(segment
+		(start 176.2525 78.74)
+		(end 177.4 78.74)
+		(width 0.14)
+		(layer "B.Cu")
+		(net "+3V3")
+	)
+	(segment
+		(start 152.745 75.4)
+		(end 172.9125 75.4)
+		(width 0.14)
+		(layer "B.Cu")
+		(net "+3V3")
+	)
+	(segment
+		(start 179.823 76.142404)
+		(end 180.09 75.875404)
+		(width 0.14)
+		(layer "B.Cu")
+		(net "+3V3")
+	)
+	(segment
+		(start 177.4 78.74)
+		(end 179.823 76.317)
+		(width 0.14)
+		(layer "B.Cu")
+		(net "+3V3")
+	)
+	(segment
+		(start 179.823 76.317)
+		(end 179.823 76.142404)
+		(width 0.14)
+		(layer "B.Cu")
+		(net "+3V3")

Commit message: updated muichiro_desk_lamp
Routing:
- added copper zone on F.Cu, net GND
Changed lines of the file:
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@@
 		(property "Value" "LOGO"
 			(at 0.75 0 0)
-			(layer "F.SilkS")
+			(layer "F.Mask")
 			(hide yes)
 			(effects
@@
 	)
 	(zone
+		(net "GND")
+		(layer "F.Cu")
+		(hatch edge 0.5)
+		(priority 1)
+		(connect_pads
+			(clearance 0.5)
+		)
+		(min_thickness 0.25)
+		(fill yes
+			(thermal_gap 0.5)
+			(thermal_bridge_width 0.5)
+			(island_removal_mode 0)
+		)
+		(polygon
+			(pts
+				(xy 133.604 29.972) (xy 201.676 32.004) (xy 203.708 140.716) (xy 128.524 140.208)
+			)
+		)
+	)
+	(zone
