File: Tamagotchi/Tamagotchi.kicad_pcb (KiCad board)
At the start: 2 copper layers, 70.1 x 85.3 mm, 18 parts, among them SW1 SW_Push, SW2 SW_Push, SW3 SW_Push, SW4 SW_Push, SW5 SW_SPDT, U1 ESP32-C3-SuperMini, U2 SSD1306

Commit message: updated Tamagotchi and muichiro_desk_lamp
Other:
- board text added: "Carson Wu Tamagotchi 19/10/2026"
- board text added: "ESP32-C3-SuperMini"
- board text added: "JLCJLCJLCJLC"
- board text added: "SSD1306"
Changed lines of the file:
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@@
 		(layer "Edge.Cuts")
+	)
+	(gr_text "ESP32-C3-SuperMini"
+		(at 126.492 120.396 90)
+		(layer "F.SilkS")
+		(effects
+			(font
+				(size 1 1)
+				(thickness 0.2)
+				(bold yes)
+			)
+			(justify left bottom)
+		)
+	)
+	(gr_text "SSD1306"
+		(at 140.208 80.772 0)
+		(layer "F.SilkS")
+		(effects
+			(font
+				(size 1.5 1.5)
+				(thickness 0.3)
+				(bold yes)
+			)
+			(justify left bottom)
+		)
+	)
+	(gr_text "Carson Wu\nTamagotchi\n19/10/2026"
+		(at 132.588 97.536 0)
+		(layer "B.SilkS")
+		(effects
+			(font
+				(size 1.5 1.5)
+				(thickness 0.3)
+				(bold yes)
+			)
+			(justify left bottom mirror)
+		)
+	)
+	(gr_text "JLCJLCJLCJLC"
+		(at 152.4 82.804 0)
+		(layer "B.SilkS")
+		(effects
+			(font
+				(size 1.5 1.5)
+				(thickness 0.3)
+				(bold yes)
+			)
+			(justify left bottom mirror)
+		)
 	)
 	(segment

Commit message: updated Tamagotchi
Parts:
- moved U1 39.9 mm to (160.0, 91.7)
- moved BT1 33.1 mm to (169.2, 111.3), turned to 180 degrees
- moved U2 16.6 mm to (134.4, 90.7)
Routing:
- net Net-(U1-GPIO0): track 34.9 -> 118.7 mm
- net Net-(U1-GPIO8): track 62.0 -> 17.8 mm
- net Net-(U1-GPIO1): track 46.5 -> 86.3 mm, vias 0 -> 1
- net Net-(U1-GPIO9): track 60.7 -> 21.4 mm
- net Net-(BT1-+): track 51.7 -> 21.2 mm, vias 1 -> 0
- net Net-(U1-GPIO2): track 44.8 -> 69.2 mm, vias 0 -> 1
- net Net-(U1-GPIO3): track 55.3 -> 68.8 mm, vias 0 -> 4
- net Net-(U1-GPIO4): track 45.0 -> 58.4 mm
- net Net-(SW5-C): track 144.2 -> 149.2 mm, vias 2 -> 4
- net GND: track 6.64 -> 2.54 mm, vias 2 -> 1
- net Net-(D1-A): track 25.2 -> 21.4 mm, vias 2 -> 0

Commit message: updated Tamagotchi and muichiro_desk_lamp
Parts:
- added REF**: MountingHole_3.2mm_M3, MountingHole:MountingHole_3.2mm_M3, F.Cu at (116.8, 99.1)
- added REF**: MountingHole_3.2mm_M3, MountingHole:MountingHole_3.2mm_M3, F.Cu at (145.3, 67.1)
- added REF**: MountingHole_3.2mm_M3, MountingHole:MountingHole_3.2mm_M3, F.Cu at (176.3, 108.7)
Routing:
- net Net-(SW5-C): track 149.2 -> 147.8 mm

Commit message: updated Tamagotchi
Routing:
- net Net-(U1-GPIO4): track 58.4 -> 59.2 mm
- net GND: vias 1 -> 2
Changed lines of the file:
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@@
 	)
 	(setup
+		(stackup
+			(layer "F.SilkS"
+				(type "Top Silk Screen")
+			)
+			(layer "F.Paste"
+				(type "Top Solder Paste")
+			)
+			(layer "F.Mask"
+				(type "Top Solder Mask")
+				(thickness 0.01)
+			)
+			(layer "F.Cu"
+				(type "copper")
+				(thickness 0.035)
+			)
+			(layer "dielectric 1"
+				(type "core")
+				(thickness 1.51)
+				(material "FR4")
+				(epsilon_r 4.5)
+				(loss_tangent 0.02)
+			)
+			(layer "B.Cu"
+				(type "copper")
+				(thickness 0.035)
+			)
+			(layer "B.Mask"
+				(type "Bottom Solder Mask")
+				(thickness 0.01)
+			)
+			(layer "B.Paste"
+				(type "Bottom Solder Paste")
+			)
+			(layer "B.SilkS"
+				(type "Bottom Silk Screen")
+			)
+			(copper_finish "None")
+			(dielectric_constraints no)
+		)
 		(pad_to_mask_clearance 0)
 		(allow_soldermask_bridges_in_footprints no)
@@
 		(capping no)
 		(filling no)
+		(zone_defaults)
 		(pcbplotparams
 			(layerselection 0x00000000_00000000_55555555_5755f5ff)
@@
 	)
 	(segment
+		(start 171.596 91.84)
+		(end 167.64 87.884)
+		(width 0.2)
+		(layer "F.Cu")
+		(net "Net-(SW5-C)")
+	)
+	(segment
 		(start 166.597244 137.668)
 		(end 160.528 137.668)
@@
 	)
 	(segment
+		(start 171.456 127.26)
+		(end 171.596 127.12)
+		(width 0.2)
+		(layer "F.Cu")
+		(net "Net-(SW5-C)")
+	)
+	(segment
 		(start 137.57816 144.48316)
 		(end 142.74384 144.48316)
@@
 	)
 	(segment
-		(start 171.256 127.06)
-		(end 171.256 91.5)
-		(width 0.2)
-		(layer "F.Cu")
-		(net "Net-(SW5-C)")
-	)
-	(segment
 		(start 169.164 131.064)
 		(end 168.656 131.572)
@@
 	)
 	(segment
-		(start 171.256 91.5)
-		(end 167.64 87.884)
+		(start 170.256 131.064)
+		(end 169.164 131.064)
 		(width 0.2)
 		(layer "F.Cu")
@@
 	)
 	(segment
-		(start 170.256 131.064)
-		(end 169.164 131.064)
+		(start 171.456 129.54)
+		(end 171.456 127.26)
 		(width 0.2)
 		(layer "F.Cu")
@@
 	)
 	(segment
-		(start 171.456 129.54)
-		(end 171.456 127.26)
+		(start 168.51 82.443634)
+		(end 168.51 87.014)
 		(width 0.2)
 		(layer "F.Cu")
@@
 	)
 	(segment
-		(start 168.51 82.443634)
-		(end 168.51 87.014)
+		(start 144.996 144.281)
+		(end 151.074 144.281)
 		(width 0.2)
 		(layer "F.Cu")
@@
 	)
 	(segment
-		(start 144.996 144.281)
-		(end 151.074 144.281)
+		(start 171.596 127.12)
+		(end 171.596 91.84)
 		(width 0.2)
 		(layer "F.Cu")
@@
 		(net "Net-(SW5-C)")
 	)
-	(segment
-		(start 171.456 127.26)
-		(end 171.256 127.06)
-		(width 0.2)
-		(layer "F.Cu")
-		(net "Net-(SW5-C)")
-	)
 	(via
 		(at 171.456 129.54)
@@
 	)
 	(segment
-		(start 151.984 139.284)
+		(start 152.4 139.7)
 		(end 151.892 139.192)
 		(width 0.2)
@@
 	)
 	(segment
-		(start 171.196 131.064)
-		(end 170.256 131.064)
+		(start 160.528 137.668)
+		(end 158.496 139.7)
 		(width 0.2)
 		(layer "B.Cu")
@@
 	)
 	(segment
-		(start 158.912 139.284)
-		(end 151.984 139.284)
+		(start 171.196 131.064)
+		(end 170.256 131.064)
 		(width 0.2)
 		(layer "B.Cu")
@@
 	)
 	(segment
-		(start 171.456 129.54)
-		(end 171.456 130.804)
+		(start 158.496 139.7)
+		(end 152.4 139.7)
 		(width 0.2)
 		(layer "B.Cu")
@@
 	)
 	(segment
-		(start 160.528 137.668)
-		(end 158.912 139.284)
+		(start 171.456 129.54)
+		(end 171.456 130.804)
 		(width 0.2)
 		(layer "B.Cu")
@@
 	)
 	(segment
-		(start 150.616529 136.744)
-		(end 142.332 136.744)
+		(start 167.17 103.594)
+		(end 167.17 120.33195)
 		(width 0.2)
 		(layer "B.Cu")
@@
 	)
 	(segment
-		(start 167.17 120.190529)
-		(end 150.616529 136.744)
+		(start 150.34195 137.16)
+		(end 142.748 137.16)
 		(width 0.2)
 		(layer "B.Cu")
@@
 	)
 	(segment
-		(start 167.17 103.594)
-		(end 167.17 120.190529)
+		(start 168.51 98.914)
+		(end 168.51 102.254)
 		(width 0.2)
 		(layer "B.Cu")
@@
 	)
 	(segment
-		(start 142.332 136.744)
-		(end 140.208 134.62)
+		(start 167.17 120.33195)
+		(end 150.34195 137.16)
 		(width 0.2)
 		(layer "B.Cu")
@@
 	)
 	(segment
-		(start 168.51 98.914)
-		(end 168.51 102.254)
+		(start 142.748 137.16)
+		(end 140.208 134.62)
 		(width 0.2)
 		(layer "B.Cu")
@@
 	)
 	(via
+		(at 139.7 138.684)
+		(size 0.8)
+		(drill 0.3)
+		(layers "F.Cu" "B.Cu")
+		(free yes)
+		(net "GND")
+	)
+	(via
 		(at 150.368 140.716)
 		(size 0.8)
@@
 	)
 	(segment
-		(start 170.856 135.132)
-		(end 169.959381 135.132)
+		(start 162.243 140.7)
+		(end 161.243 139.7)
+		(width 0.2)
+		(layer "F.Cu")
+		(net "Net-(U1-GPIO4)")
+	)
+	(segment
+		(start 171.196 126.954315)
+		(end 170.756 127.394315)
+		(width 0.2)
+		(layer "F.Cu")
+		(net "Net-(U1-GPIO4)")
+	)
+	(segment
+		(start 167.64 90.424)
+		(end 171.196 93.98)
 		(width 0.2)
 		(layer "F.Cu")
@@
 	)
 	(segment
-		(start 162.243 140.7)
-		(end 161.243 139.7)
+		(start 170.756 127.394315)
+		(end 170.756 129.82995)
 		(width 0.2)
 		(layer "F.Cu")
@@
 	)
 	(segment
-		(start 164.391381 140.7)
-		(end 162.243 140.7)
+		(start 171.196 135.132)
+		(end 169.959381 135.132)
 		(width 0.2)
 		(layer "F.Cu")
@@
 	)
 	(segment
-		(start 170.856 93.64)
-		(end 170.856 135.132)
+		(start 171.196 130.26995)
+		(end 171.196 135.132)
 		(width 0.2)
 		(layer "F.Cu")
@@
 	)
 	(segment
-		(start 167.64 90.424)
-		(end 170.856 93.64)
+		(start 170.756 129.82995)
+		(end 171.196 130.26995)
+		(width 0.2)
+		(layer "F.Cu")
+		(net "Net-(U1-GPIO4)")
+	)
+	(segment
+		(start 164.391381 140.7)
+		(end 162.243 140.7)
+		(width 0.2)
+		(layer "F.Cu")
+		(net "Net-(U1-GPIO4)")
+	)
+	(segment
+		(start 171.196 93.98)
+		(end 171.196 126.954315)
 		(width 0.2)
 		(layer "F.Cu")
