File: muichiro_desk_lamp/PCB/muichiro_desk_lamp.kicad_pcb (KiCad board)
At the start: 2 copper layers, 58.3 x 70.7 mm, 14 parts, among them J1 Conn_01x03_Pin, J2 Conn_01x08_Socket, J3 Conn_01x08_Socket

Commit message: updated Tamagotchi and muichiro_desk_lamp
Other:
- board text added: "LED (Blue)"
- board text removed: "Carson Wu muichiro_desk_lamp 19/10/2026"
- board text removed: "LED (Green)"
Changed lines of the file:
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@@
-		)
-	)
-	(gr_text "Carson Wu\nmuichiro_desk_lamp\n19/10/2026"
-		(at 180.34 57.404 0)
-		(layer "B.SilkS")
-		(effects
-			(font
-				(size 1.524 1.524)
-				(thickness 0.3048)
-				(bold yes)
-			)
-			(justify left bottom mirror)
 		)
 	)
@@
 		)
 	)
-	(gr_text "LED\n(Green)"
+	(gr_text "LED\n(Blue)"
 		(at 186.52 113.5 0)
 		(layer "B.SilkS")
